Commit message: 修正部署份 URDF 的关节符号，统一 base 惯量，新增模型一致性检查
问题：Imgo2_deploy 的 12 个腿部关节 axis 全部与训练份相反（q_部署 = -q_训练，限位镜像）。核对其三条推理链路（rl_real_imgo2.cpp 走 Unitree SDK、rl_sim.cpp 走 ROS 控制器、rl_sim_mujoco.cpp 走 MJCF）均无任何符号取反，只有 joint_mapping 索引置换，robot_control.yaml 也只做控制器到关节名映射，即无补偿；读该 URDF 的只有 Gazebo/ROS。

修改：部署份改为训练份约定（24 行：12 axis + 8 限位 + base 惯量块）。FK 验证对录制数据恒等 RMSE 由 0.057-0.118 m 降到 0.0001-0.0016 m，与训练份一致——即修正前该模型无法重现真机录制动作。base 质量按确认真值 5.53394020 统一：imgo2_description/urdf/imgo2.urdf 原为 6.53394020 却带 3.5339 那份惯量（质量与惯量不自洽，比值 1.566 恰为 5.5339/3.5339），一并改为规范块。

核实 imgo2_description 两个 URDF 的符号与限位本来即与训练份一致，且都能重现录制数据，故采集数据无问题；xacro/robot.xacro 直接 include urdf/imgo2_description.urdf，common/leg.xacro 与 urdf/imgo2.urdf 全工作区无人引用。

新增 scripts/tools/check_model_sync.py（纯标准库）：按逻辑关节名（与腿序无关，故容忍 imgo2_description 的有意腿序差异）比对四份 URDF 的轴/限位、base 惯量、三份共用网格，并对每份做 FK。本机四项全通过；已用『故意翻回符号』的负向测试确认可报错，恢复后 sha256 不变。

File: Imgo2_deploy/robot_description/imgo2_urdf/urdf/imgo2.urdf (robot description, URDF)
Before this commit: robot Imgo2, 17 links, 16 joints
Links:
- link base: mass 3.53394020 -> 5.53394020
Joints:
- joint FL_hip_joint: axis -1 0 0 -> 1 0 0
- joint FL_shank_joint: axis 0 -1 0 -> 0 1 0; limit lower=0.733 upper=3.0 effort=23.7 velocity=30.1 -> lower=-3.0 upper=-0.733 effort=23.7 velocity=30.1
- joint FL_thigh_joint: axis 0 -1 0 -> 0 1 0; limit lower=-2.87 upper=0.9 effort=23.7 velocity=30.1 -> lower=-0.9 upper=2.87 effort=23.7 velocity=30.1
- joint FR_hip_joint: axis -1 0 0 -> 1 0 0
- joint FR_shank_joint: axis 0 -1 0 -> 0 1 0; limit lower=0.733 upper=3.0 effort=23.7 velocity=30.1 -> lower=-3.0 upper=-0.733 effort=23.7 velocity=30.1
- joint FR_thigh_joint: axis 0 -1 0 -> 0 1 0; limit lower=-2.87 upper=0.9 effort=23.7 velocity=30.1 -> lower=-0.9 upper=2.87 effort=23.7 velocity=30.1
- joint RL_hip_joint: axis -1 0 0 -> 1 0 0
- joint RL_shank_joint: axis 0 -1 0 -> 0 1 0; limit lower=0.733 upper=3.0 effort=23.7 velocity=30.1 -> lower=-3.0 upper=-0.733 effort=23.7 velocity=30.1
- joint RL_thigh_joint: axis 0 -1 0 -> 0 1 0; limit lower=-2.87 upper=0.9 effort=23.7 velocity=30.1 -> lower=-0.9 upper=2.87 effort=23.7 velocity=30.1
- joint RR_hip_joint: axis -1 0 0 -> 1 0 0
- joint RR_shank_joint: axis 0 -1 0 -> 0 1 0; limit lower=0.733 upper=3.0 effort=23.7 velocity=30.1 -> lower=-3.0 upper=-0.733 effort=23.7 velocity=30.1
- joint RR_thigh_joint: axis 0 -1 0 -> 0 1 0; limit lower=-2.87 upper=0.9 effort=23.7 velocity=30.1 -> lower=-0.9 upper=2.87 effort=23.7 velocity=30.1

File: imgo2_description/urdf/imgo2.urdf (robot description, URDF)
Before this commit: robot Imgo2, 17 links, 16 joints
Links:
- link base: mass 6.53394020 -> 5.53394020

Commit message: 按用户决定把四份模型的物理参数全部对齐到训练侧，并扩展一致性检查
用户决定「都使用训练侧的参数」，足端碰撞圆柱也「保持训练侧」。据此：

- Imgo2_deploy 的足端 CoM/惯量与后腿 shank/thigh 惯量非对角项（五份模型
  中的唯一异类）改为训练侧，共替换 8 个 inertial 块。
- 四份 URDF 的足端碰撞圆柱长度由 2 对 3 的分布统一为训练侧的 0.01。
- Imgo2_deploy 的质量值尾随空格清理。
- imgo2_description 的两个 URDF 只改了足端碰撞圆柱（0.02 -> 0.01），
  它们的关节与惯量本来就与训练侧一致。

结果：四份完整 URDF 按逻辑 link 名比对的物理指纹完全一致
（aae81e7301f5），Imgo2_deploy 与训练份现仅差 4 个不影响物理的
<material> 块。

check_model_sync.py 新增第 2 项「逐 link 质量/质心/惯量/碰撞几何」检查并
重新编号，第 3 项起顺延；本机五项全通过，并新增第 2 次负向测试（只改足端
CoM、不动关节）确认能报错，恢复后 sha256 不变。

README 的代码导航、离线检查说明、状态表与维护记录，以及 AGENTS.md 的
「模型与资源路径」一节同步更新。未运行 Isaac Lab 或 Gazebo。

File: Imgo2_deploy/robot_description/imgo2_urdf/urdf/imgo2.urdf (robot description, URDF)
Before this commit: robot Imgo2, 17 links, 16 joints
Links:
- link FL_FOOT: geometry collision cylinder length=0.01 radius=0.0155; collision sphere radius=0.022
- link FL_SHANK: mass 0.09561741  -> 0.09561741
- link FL_THIGH: mass 0.96995719  -> 0.96995719
- link FR_FOOT: geometry collision cylinder length=0.01 radius=0.0155; collision sphere radius=0.022
- link FR_SHANK: mass 0.09561741  -> 0.09561741
- link FR_THIGH: mass 0.96995719  -> 0.96995719
- link RL_FOOT: geometry collision cylinder length=0.01 radius=0.0155; collision sphere radius=0.022
- link RL_SHANK: mass 0.09561741  -> 0.09561741
- link RL_THIGH: mass 0.96995719  -> 0.96995719
- link RR_FOOT: geometry collision cylinder length=0.01 radius=0.0155; collision sphere radius=0.022
- link RR_SHANK: mass 0.09561741  -> 0.09561741
- link RR_THIGH: mass 0.96995719  -> 0.96995719

File: imgo2_description/urdf/imgo2.urdf (robot description, URDF)
Before this commit: robot Imgo2, 17 links, 16 joints
Links:
- link FL_FOOT: geometry collision cylinder length=0.01 radius=0.0155; collision sphere radius=0.022
- link FR_FOOT: geometry collision cylinder length=0.01 radius=0.0155; collision sphere radius=0.022
- link RL_FOOT: geometry collision cylinder length=0.01 radius=0.0155; collision sphere radius=0.022
- link RR_FOOT: geometry collision cylinder length=0.01 radius=0.0155; collision sphere radius=0.022

File: imgo2_description/urdf/imgo2_description.urdf (robot description, URDF)
Before this commit: robot Imgo2, 17 links, 16 joints
Links:
- link LF_FOOT: geometry collision cylinder length=0.01 radius=0.0155; collision sphere radius=0.022
- link LH_FOOT: geometry collision cylinder length=0.01 radius=0.0155; collision sphere radius=0.022
- link RF_FOOT: geometry collision cylinder length=0.01 radius=0.0155; collision sphere radius=0.022
- link RH_FOOT: geometry collision cylinder length=0.01 radius=0.0155; collision sphere radius=0.022
