Commit message: 模型统一阶段①②：imgo2_description 命名/网格统一 + xacro 模块化 + 生成物入库
按用户决定执行（D1 FL/FR/RL/RR；D2 Gazebo 模块留在 description；D3 生成物入库；
D4 删冗余、git 兜底；D5 插件暂不处理）。

模型源
- 新增 xacro/core.xacro：由训练 URDF 抽出 17 link / 16 joint（含 <robot> 包裹以便
  xacro:include），作为物理唯一准绳；不含 Gazebo / transmission / IMU
- 新增 xacro/transmission.xacro：修正旧宏 params="name" 却使用 ${prefix} 的错误，
  按 prefix 生成 3 个 transmission；旧文件从未被 include，是死代码
- 新增 xacro/gazebo.xacro：2 个插件块 + 17 个 per-link 接触块，link 名改为 FL 命名
- 新增 xacro/imu.xacro；重写 xacro/robot.xacro 为组装入口，开关 transmission / gazebo /
  imu，默认全 false
- meshes 改名 LF_hip→FL_hip、LH_hip→RL_hip、RF_hip→FR_hip、RH_hip→RR_hip、
  L_calf→L_shank、R_calf→R_shank（内容逐字节不变；四份网格指纹统一为 8dc5b5995a11）

生成物（入库，勿手改）
- urdf/imgo2.urdf：core only，17 link / 16 joint，无附加块
- urdf/imgo2.gazebo.urdf：core + transmission 12 + gazebo 21 + base_imu

删除
- urdf/imgo2_description.urdf（被 imgo2.gazebo.urdf 取代）
- xacro/common/（5 个文件：gazebo/imu/transmission 已被 xacro/*.xacro 取代，
  leg.xacro 引用仓库外的 legged_unitree_description，materials.xacro 无人引用）

配套
- empty_world.launch 显式传 transmission:=true gazebo:=true imu:=true，并注明仍依赖
  不在仓库的 legged_common / legged_gazebo（DEPLOY-05）
- CMakeLists.txt 安装目录补 xacro mjcf
- check_model_sync.py：登记两份生成物（Gazebo 份允许 base_imu）、网格集纳入
  imgo2_description/meshes、去掉已无用的 DESC_TO_TRAIN、更新提示与汇总文案
- check_amp_joint_order.py：默认模型改为 imgo2_description/urdf/imgo2.urdf，
  FK 段改用 audit 自带的跨腿交换对照

验证
- check_model_sync.py 五项全 PASS：4 份已登记 URDF 的关节轴/限位、17 link 质量/质心/
  惯量/碰撞、base 规范值全一致，网格四份逐字节相同，FK 恒等 RMSE 0.00214 m / 交换 0.22470 m
- check_amp_joint_order.py 三项全 PASS，数值与统一前完全一致（0.00107/0.00214 m、0.22491、
  0.0191 对 0.1339 rad、r 0.9546 对 0.2317；新 URDF hash c4f14273959e94c1）
- 生成物与训练 URDF 结构等价：links/joints 集合相同，轴/限位/origin/惯量/碰撞逐项相同
- xacro 重跑两次与入库文件逐字节一致（生成物可复现）
- 负向测试：把首个 hip 轴改为 -1 0 0 → 报 2 条 FAIL（关节轴不同、FK 退化到 0.02910 m），
  恢复后 SHA256 不变
- check_asset_paths.py PASS；git ls-files -i -c --exclude-standard 为空

未做：消费者切换、MJCF 归位、删除镜像副本（见 README MODEL-02）。未运行训练/GUI/ROS/真机。

File: imgo2_description/urdf/imgo2.gazebo.urdf (robot description, URDF)
Before this commit: robot Imgo2, 17 links, 16 joints
Links:
- added link base_imu, mass 0.01; visual box size=0.015 0.015 0.004
Joints:
- added joint base_imu_joint: type fixed, parent base, child base_imu, origin xyz=0 0 0 rpy=0 0 0

File: imgo2_description/xacro/robot.xacro (robot description, xacro)
@@ -1,7 +1,32 @@
 <?xml version="1.0"?>
-<robot name="imgo2_description" xmlns:xacro="http://www.ros.org/wiki/xacro">
-    <xacro:include filename="$(find imgo2_description)/urdf/imgo2_description.urdf"/>
-    <xacro:include filename="$(find imgo2_description)/xacro/common/gazebo.xacro"/>
-    <xacro:include filename="$(find imgo2_description)/xacro/common/imu.xacro"/>
-    <xacro:IMU connected_to="base" imu_name="base_imu" xyz="0. 0. 0." rpy="0. 0. 0."/>
+<!-- Imgo2 模型组装入口（imgo2_description 是模型的唯一源）。
+     用法：
+       xacro robot.xacro                                            # 纯 URDF：RL / 非 Gazebo 消费者
+       xacro robot.xacro transmission:=true gazebo:=true imu:=true   # Gazebo / ROS 链路
+     开关默认全 false，所以不带参数时只输出 core.xacro 的内核（links + joints），
+     与训练侧 URDF 等价。
+     生成物（已入库，勿手改；改了要重新生成并跑校验）：
+       ../urdf/imgo2.urdf          <- core only
+       ../urdf/imgo2.gazebo.urdf   <- core + transmission + gazebo + imu
+-->
+<robot name="Imgo2" xmlns:xacro="http://www.ros.org/wiki/xacro">
+    <xacro:arg name="transmission" default="false"/>
+    <xacro:arg name="gazebo" default="false"/>
+    <xacro:arg name="imu" default="false"/>
+    <!-- 内核：物理参数唯一准绳 -->
+    <xacro:include filename="core.xacro"/>
+    <xacro:if value="$(arg transmission)">
+        <xacro:include filename="transmission.xacro"/>
+        <xacro:leg_transmission prefix="FL"/>
+        <xacro:leg_transmission prefix="FR"/>
+        <xacro:leg_transmission prefix="RL"/>
+        <xacro:leg_transmission prefix="RR"/>
+    </xacro:if>
+    <xacro:if value="$(arg gazebo)">
+        <xacro:include filename="gazebo.xacro"/>
+    </xacro:if>
+    <xacro:if value="$(arg imu)">
+        <xacro:include filename="imu.xacro"/>
+        <xacro:IMU connected_to="base" imu_name="base_imu" xyz="0 0 0" rpy="0 0 0"/>
+    </xacro:if>
 </robot>

Commit message: 打通 Gazebo/ROS 2 链路：改用 gazebo_ros2_control（DEPLOY-05）
原先 Gazebo 链路挂的是上游 ROS 1 的 liblegged_hw_sim.so（gazebo_ros_control），仓库里没有、
本机 ROS 2 也没有，controller spawner 找不到 controller_manager。照参考项目改为
ROS 2 gazebo_ros2_control（本机 Humble 自带 0.4.10）：

- imgo2_description/xacro/gazebo.xacro：加 IMU 传感器（libgazebo_ros_imu_sensor.so，挂 base_imu，
  remap ~/out:=imu）、<ros2_control name="GazeboSystem">（12 关节 effort 命令 + position/velocity/
  effort 状态）、libgazebo_ros2_control.so 插件；删掉不可用的 liblegged_hw_sim 与 ROS1 p3d。
- 新增 imgo2_description/config/robot_control_ros2.yaml：joint_state_broadcaster +
  robot_joint_controller/RobotJointControllerGroup（仓库内控制器，由 rl_sim 自己 spawn）。
- imgo2_description 做成标准 ROS 2 包：ament CMakeLists（装 config/launch/meshes/urdf/xacro/mjcf）、
  package.ros1.xml + package.ros2.xml，package.xml 由 build.sh 按 ROS_DISTRO 换成软链；
  build.sh 包扫描改 find -L src；imgo2_deploy/src/imgo2_description 为指向仓库根的软链（不复制模型）。
- core.xacro/robot.xacro：网格前缀改为 xacro 属性 mesh_prefix —— 纯 URDF 仍 ../meshes/（重生成后
  与原文件逐字节相同），gazebo:=true 时用 package://imgo2_description/meshes/；
  check_model_sync.py 的网格引用检查两种写法都认。
- launch/gazebo.launch.py 重写：自己起 gzserver/gzclient（不用 gazebo_ros 自带 launch，本机实测它
  起的 gzserver 没加载 factory 插件）、加 wname/gui 参数、把 URDF 里的 package://imgo2_description
  换成实际 share 路径并压成单行写到临时文件、用 -file spawn、spawn 完再起 joint_state_broadcaster。

两个实测坑（都写进文档）：
1. gazebo_ros2_control 0.4.x 的 <parameters> 只认真实文件路径，package:// 或相对路径都会让插件
   Load 抛异常；
2. URDF 以 --param robot_description:=<xml> 交给 controller_manager 时带换行会报
   "Couldn't parse parameter override rule"，CM 拿不到 URDF、控制器起不来。

验证：bash build.sh 4 个包全过（rl_sim 43.8 MB，POLICY_DIR 指向本仓库 policy，
share/imgo2_description/config/robot_control_ros2.yaml 就位）；无头单次调用内 spawn 成功、网格 0 报错、
节点 /gazebo_ros2_control 与 /imu_plugin 出现、joint_state_broadcaster active、/joint_states 与 /imu
发布、rl_sim 经 /joy 注入 A→RB+DPadUp 后打印 "RL Controller [ppo]"（进入键 1 的 PPO 闭环）；
check_model_sync/check_asset_paths/check_amp_joint_order 仍全 PASS。

未验证：GUI 画面与步态观感（本机 DISPLAY=:1 建 GL 上下文失败）、himloco/AMP 长时间行为、真机。
文档：新增 docs/gazebo_ros2_bringup_2026-09-17.md；README §6.2/DEPLOY-05/维护记录、AGENTS 模型章节同步。

File: imgo2_description/urdf/imgo2.gazebo.urdf (robot description, URDF)
Before this commit: robot Imgo2, 18 links, 17 joints
Links:
- link FL_FOOT: geometry collision cylinder length=0.01 radius=0.0155; collision sphere radius=0.022
- link FL_HIP: geometry collision cylinder length=0.041 radius=0.048; visual mesh filename=package://imgo2_description/meshes/FL_hip.STL scale=1 1 1
- link FL_SHANK: geometry collision cylinder length=0.08 radius=0.012; collision cylinder length=0.1 radius=0.012
- link FL_THIGH: geometry collision box size=0.06 0.032 0.22; collision cylinder length=0.046 radius=0.048
- link FR_FOOT: geometry collision cylinder length=0.01 radius=0.0155; collision sphere radius=0.022
- link FR_HIP: geometry collision cylinder length=0.041 radius=0.048; visual mesh filename=package://imgo2_description/meshes/FR_hip.STL scale=1 1 1
- link FR_SHANK: geometry collision cylinder length=0.08 radius=0.012; collision cylinder length=0.1 radius=0.012
- link FR_THIGH: geometry collision box size=0.06 0.032 0.22; collision cylinder length=0.046 radius=0.048
- link RL_FOOT: geometry collision cylinder length=0.01 radius=0.0155; collision sphere radius=0.022
- link RL_HIP: geometry collision cylinder length=0.041 radius=0.048; visual mesh filename=package://imgo2_description/meshes/RL_hip.STL scale=1 1 1
- link RL_SHANK: geometry collision cylinder length=0.08 radius=0.012; collision cylinder length=0.1 radius=0.012
- link RL_THIGH: geometry collision box size=0.06 0.032 0.22; collision cylinder length=0.046 radius=0.048
- link RR_FOOT: geometry collision cylinder length=0.01 radius=0.0155; collision sphere radius=0.022
- link RR_HIP: geometry collision cylinder length=0.041 radius=0.048; visual mesh filename=package://imgo2_description/meshes/RR_hip.STL scale=1 1 1
- link RR_SHANK: geometry collision cylinder length=0.08 radius=0.012; collision cylinder length=0.1 radius=0.012
- link RR_THIGH: geometry collision box size=0.06 0.032 0.22; collision cylinder length=0.046 radius=0.048
- link base: geometry collision box size=0.018 0.012 0.018; collision box size=0.018 0.012 0.018

File: imgo2_description/xacro/core.xacro (robot description, xacro)
@@ -4,5 +4,6 @@
      命名与训练侧一致：FL/FR/RL/RR，关节 FL_hip_joint / FL_thigh_joint / FL_shank_joint，
      足端固定关节 FL_Ankle，link 名 base / FL_HIP / FL_THIGH / FL_SHANK / FL_FOOT。
-     网格相对于 <repo>/imgo2_description/meshes/ 解析。 -->
+     网格前缀由 xacro 属性 mesh_prefix 决定（robot.xacro 按 gazebo 开关设为 ../meshes/ 或
+      package://imgo2_description/meshes/），故本文件必须经 robot.xacro 组装。 -->
 <robot xmlns:xacro="http://www.ros.org/wiki/xacro">
 <link name="base">
@@ -17,5 +18,5 @@
             <origin rpy="0 0 0" xyz="0 0 0.0"/>
             <geometry>
-                <mesh filename="../meshes/base.STL"/>
+                <mesh filename="${mesh_prefix}base.STL"/>
             </geometry>
         </visual>
@@ -64,5 +65,5 @@
         <visual>
             <geometry>
-                <mesh filename="../meshes/FL_hip.STL" scale="1 1 1"/>
+                <mesh filename="${mesh_prefix}FL_hip.STL" scale="1 1 1"/>
             </geometry>
         </visual>
@@ -91,5 +92,5 @@
         <visual>
             <geometry>
-                <mesh filename="../meshes/L_thigh.STL"/>
+                <mesh filename="${mesh_prefix}L_thigh.STL"/>
             </geometry>
         </visual>
@@ -124,5 +125,5 @@
         <visual>
             <geometry>
-                <mesh filename="../meshes/L_shank.STL"/>
+                <mesh filename="${mesh_prefix}L_shank.STL"/>
             </geometry>
         </visual>
@@ -155,5 +156,5 @@
         <visual>
             <geometry>
-                <mesh filename="../meshes/foot.STL"/>
+                <mesh filename="${mesh_prefix}foot.STL"/>
             </geometry>
         </visual>
@@ -187,5 +188,5 @@
         <visual>
             <geometry>
-                <mesh filename="../meshes/FR_hip.STL" scale="1 1 1"/>
+                <mesh filename="${mesh_prefix}FR_hip.STL" scale="1 1 1"/>
             </geometry>
         </visual>
@@ -214,5 +215,5 @@
         <visual>
             <geometry>
-                <mesh filename="../meshes/R_thigh.STL"/>
+                <mesh filename="${mesh_prefix}R_thigh.STL"/>
             </geometry>
         </visual>
@@ -247,5 +248,5 @@
         <visual>
             <geometry>
-                <mesh filename="../meshes/R_shank.STL"/>
+                <mesh filename="${mesh_prefix}R_shank.STL"/>
             </geometry>
         </visual>
@@ -278,5 +279,5 @@
         <visual>
             <geometry>
-                <mesh filename="../meshes/foot.STL"/>
+                <mesh filename="${mesh_prefix}foot.STL"/>
             </geometry>
         </visual>
@@ -310,5 +311,5 @@
         <visual>
             <geometry>
-                <mesh filename="../meshes/RL_hip.STL" scale="1 1 1"/>
+                <mesh filename="${mesh_prefix}RL_hip.STL" scale="1 1 1"/>
             </geometry>
         </visual>
@@ -337,5 +338,5 @@
         <visual>
             <geometry>
-                <mesh filename="../meshes/L_thigh.STL"/>
+                <mesh filename="${mesh_prefix}L_thigh.STL"/>
             </geometry>
         </visual>
@@ -370,5 +371,5 @@
         <visual>
             <geometry>
-                <mesh filename="../meshes/L_shank.STL"/>
+                <mesh filename="${mesh_prefix}L_shank.STL"/>
             </geometry>
         </visual>
@@ -401,5 +402,5 @@
         <visual>
             <geometry>
-                <mesh filename="../meshes/foot.STL"/>
+                <mesh filename="${mesh_prefix}foot.STL"/>
             </geometry>
         </visual>
@@ -433,5 +434,5 @@
         <visual>
             <geometry>
-                <mesh filename="../meshes/RR_hip.STL" scale="1 1 1"/>
+                <mesh filename="${mesh_prefix}RR_hip.STL" scale="1 1 1"/>
             </geometry>
         </visual>
@@ -460,5 +461,5 @@
         <visual>
             <geometry>
-                <mesh filename="../meshes/R_thigh.STL"/>
+                <mesh filename="${mesh_prefix}R_thigh.STL"/>
             </geometry>
         </visual>
@@ -493,5 +494,5 @@
         <visual>
             <geometry>
-                <mesh filename="../meshes/R_shank.STL"/>
+                <mesh filename="${mesh_prefix}R_shank.STL"/>
             </geometry>
         </visual>
@@ -524,5 +525,5 @@
         <visual>
             <geometry>
-                <mesh filename="../meshes/foot.STL"/>
+                <mesh filename="${mesh_prefix}foot.STL"/>
             </geometry>
         </visual>

File: imgo2_description/xacro/gazebo.xacro (robot description, xacro)
@@ -1,28 +1,76 @@
 <?xml version="1.0"?>
-<!-- Gazebo 专用内容：插件 + 按 link 的摩擦/接触参数。
-     只在组装 Gazebo 模型时包含（xacro/robot.xacro 的 gazebo:=true）。
+<!-- Gazebo 专用内容：IMU 传感器 + ros2_control 硬件接口 + gazebo_ros2_control 插件
+     + 按 link 的摩擦/接触参数。只在组装 Gazebo 模型时包含（xacro/robot.xacro 的
+     gazebo:=true，IMU 传感器还需要 imu:=true）。
      这些标签对 Isaac Lab / MuJoCo 无意义，故从 core.xacro 独立出来。
-     插件 liblegged_hw_sim.so 不在仓库内（见 README DEPLOY-05）。 -->
+     2026-09-17 按参考项目 ~/RL/sim2sim/Imgo2_deploy/imgo2_description/xacro/gazebo.xacro
+     对齐：旧版走 ROS1 的 `liblegged_hw_sim.so`（gazebo_ros_control + EffortJointInterface），
+     该库不在仓库内、本机也没有；现改走 ROS 2 的 `gazebo_ros2_control`（Humble 自带
+     /opt/ros/humble/lib/libgazebo_ros2_control.so），控制器是仓库内的
+     robot_joint_controller/RobotJointControllerGroup，由 rl_sim 启动。 -->
 <robot xmlns:xacro="http://www.ros.org/wiki/xacro">
-    <!-- ros_control 与地面真值插件 -->
+    <xacro:property name="hip_torque_max" value="23.7"/>
+    <xacro:property name="thigh_torque_max" value="23.7"/>
+    <xacro:property name="shank_torque_max" value="23.7"/>
+    <!-- IMU：rl_sim 订阅 /imu（sensor_msgs/Imu）。挂 base_imu（imu.xacro 生成）。 -->
+    <xacro:if value="$(arg imu)">
+    <gazebo reference="base_imu">
+        <sensor name="imu_sensor" type="imu">
+            <plugin filename="libgazebo_ros_imu_sensor.so" name="imu_plugin">
+                <ros>
+                    <namespace>/</namespace>
+                    <remapping>~/out:=imu</remapping>
+                </ros>
+                <initial_orientation_as_reference>false</initial_orientation_as_reference>
+            </plugin>
+            <always_on>true</always_on>
+            <update_rate>100</update_rate>
+            <visualize>true</visualize>
+            <imu>
+                <angular_velocity>
+                    <x><noise type="gaussian"><mean>0.0</mean><stddev>2e-4</stddev><bias_mean>0.0000075</bias_mean><bias_stddev>0.0000008</bias_stddev></noise></x>
+                    <y><noise type="gaussian"><mean>0.0</mean><stddev>2e-4</stddev><bias_mean>0.0000075</bias_mean><bias_stddev>0.0000008</bias_stddev></noise></y>
+                    <z><noise type="gaussian"><mean>0.0</mean><stddev>2e-4</stddev><bias_mean>0.0000075</bias_mean><bias_stddev>0.0000008</bias_stddev></noise></z>
+                </angular_velocity>
+                <linear_acceleration>
+                    <x><noise type="gaussian"><mean>0.0</mean><stddev>1.7e-2</stddev><bias_mean>0.1</bias_mean><bias_stddev>0.001</bias_stddev></noise></x>
+                    <y><noise type="gaussian"><mean>0.0</mean><stddev>1.7e-2</stddev><bias_mean>0.1</bias_mean><bias_stddev>0.001</bias_stddev></noise></y>
+                    <z><noise type="gaussian"><mean>0.0</mean><stddev>1.7e-2</stddev><bias_mean>0.1</bias_mean><bias_stddev>0.001</bias_stddev></noise></z>
+                </linear_acceleration>
+            </imu>
+        </sensor>
+    </gazebo>
+    </xacro:if>
+    <!-- ros2_control 硬件：gazebo_ros2_control 的 GazeboSystem，力矩命令 + 位置/速度/力矩状态 -->
+    <ros2_control name="GazeboSystem" type="system">
+        <hardware>
+            <plugin>gazebo_ros2_control/GazeboSystem</plugin>
+        </hardware>
+        <xacro:macro name="joint_interface" params="joint_name torque_limit">
+            <joint name="${joint_name}">
+                <command_interface name="effort">
+                    <param name="min">-${torque_limit}</param>
+                    <param name="max">${torque_limit}</param>
+                </command_interface>
+                <state_interface name="position"/>
+                <state_interface name="velocity"/>
+                <state_interface name="effort"/>
+            </joint>
+        </xacro:macro>
+        <xacro:macro name="leg_joints" params="prefix">
+            <xacro:joint_interface joint_name="${prefix}_hip_joint" torque_limit="${hip_torque_max}"/>
+            <xacro:joint_interface joint_name="${prefix}_thigh_joint" torque_limit="${thigh_torque_max}"/>
+            <xacro:joint_interface joint_name="${prefix}_shank_joint" torque_limit="${shank_torque_max}"/>
+        </xacro:macro>
+        <xacro:leg_joints prefix="FL"/>
+        <xacro:leg_joints prefix="FR"/>
+        <xacro:leg_joints prefix="RL"/>
+        <xacro:leg_joints prefix="RR"/>
+    </ros2_control>
     <gazebo>
-            <plugin name="gazebo_ros_control" filename="liblegged_hw_sim.so">
-                <robotNamespace>/</robotNamespace>
-                <robotParam>legged_robot_description</robotParam>
-                <robotSimType>legged_gazebo/LeggedHWSim</robotSimType>
-            </plugin>
-        </gazebo>
-    <gazebo>
-            <plugin name="p3d_base_controller" filename="libgazebo_ros_p3d.so">
-                <alwaysOn>true</alwaysOn>
-                <updateRate>1000.0</updateRate>
-                <bodyName>base</bodyName>
-                <topicName>ground_truth/state</topicName>
-                <gaussianNoise>0</gaussianNoise>
-                <frameName>world</frameName>
-                <xyzOffsets>0 0 0</xyzOffsets>
-                <rpyOffsets>0 0 0</rpyOffsets>
-            </plugin>
-        </gazebo>
+        <plugin name="gazebo_ros2_control" filename="libgazebo_ros2_control.so">
+            <parameters>package://imgo2_description/config/robot_control_ros2.yaml</parameters>
+        </plugin>
+    </gazebo>
     <!-- 按 link 的 Gazebo 接触参数（mu1/mu2/kp/kd/self_collide） -->
     <gazebo reference="base">

File: imgo2_description/xacro/robot.xacro (robot description, xacro)
@@ -15,4 +15,13 @@
     <xacro:arg name="imu" default="false"/>
     <!-- 内核：物理参数唯一准绳 -->
+    <!-- 网格前缀：纯 URDF 用相对路径 ../meshes/（相对 urdf/ 目录）；Gazebo 组装改用
+         package://imgo2_description/meshes/ —— Gazebo 经 ament 解析，这样即使 spawn 时
+         只把 URDF 文本发过去（-topic）也能找到网格，不依赖文件所在目录。 -->
+    <xacro:if value="$(arg gazebo)">
+        <xacro:property name="mesh_prefix" value="package://imgo2_description/meshes/"/>
+    </xacro:if>
+    <xacro:unless value="$(arg gazebo)">
+        <xacro:property name="mesh_prefix" value="../meshes/"/>
+    </xacro:unless>
     <xacro:include filename="core.xacro"/>
     <xacro:if value="$(arg transmission)">
