Commit message: wip(cart): 车斗配重/轮径重构（进行中）+ 工具与测试同步
本提交由用户要求「提交当前改动并 push」时落盘，内容是**同一工作区另一会话**正在进行的
小车模型重构，不是本轮 CE Net 的改动（那部分已在 212871f / ed2c973）。

现状（以源码为准）：
- `imgo2_description/cart/cart.urdf`：车斗 + **可调重物块**，轮径 0.08 → **0.03**；
- 新增 `imgo2_rl/source/imgo2_rl/imgo2_rl/assets/cart_mass.py`：由「整车总重」解析出
  合并刚体的质量 / CoM 高度 / 关于 CoM 的惯量（只改质量会让动力学不自洽）；
- `assets/cart_model.py`：读 URDF 的几何/惯量（stdlib 解析），供质量施加使用；
- `upper_mdp.py`：`initial_cart_mass` 10.0 → **3.0**（车斗 0.8 + 4×0.05 轮 + 重物块 2.0）、
  `wheel_radius` 0.08 → **0.03**、`initial_wheel_damping` 0.032 → **0.0045**（按 r² 重标定，
  保持等效滚阻 ≈ 4·damping/r²·v ≈ 20·v N）；
- `upper_env_cfg.py`：`wheel_damping_range` (0.008, 0.032) → **(0.001125, 0.0045)**；
- `scripts/towing/play_towing_test.py`：质量改到 host buffer 上按环境写入（与训练侧同做法）；
- `scripts/tools/tow_clearance.py`、`test_cart_coast_metrics.py`、`test_towing_play_test.py`、
  `test_towing_tow_clearance.py`、`test_towing_tow_metrics.py` 同步。

⚠ **WIP，未完成**：此刻 `pytest imgo2_rl/tests -q` ⇒ 665 passed, 4 skipped, **8 failed**：
- `test_towing_play_test.py`：`test_dry_run_plan_lines`、`test_mass_scaling_happens_on_host_buffer`、
  `MassScalingTests` 3 项（质量缩放接口改造尚未收尾）；
- `test_towing_upper_rl_contract.py`：min_clearance 文档表/阈值公式/reset 事件 3 项
  （挂点与表面常量随新小车几何变化，文档表尚未同步）。
CE Net 与本轮 mask 改动相关的测试全绿（见前两个提交）。README/docs 尚未记录本次小车重构。

File: imgo2_description/cart/cart.urdf (robot description, URDF)
Before this commit: robot passive_cart, 6 links, 5 joints
Links:
- added link ballast, mass 2.0; collision box size=0.3 0.3 0.3; visual box size=0.3 0.3 0.3
- link base_link: mass 8.4 -> 0.8; geometry collision box size=0.6 0.45 0.02; visual box size=0.6 0.45 0.02
- link wheel_fl: mass 0.4 -> 0.05; geometry collision cylinder length=0.04 radius=0.03; visual cylinder length=0.04 radius=0.03
- link wheel_fr: mass 0.4 -> 0.05; geometry collision cylinder length=0.04 radius=0.03; visual cylinder length=0.04 radius=0.03
- link wheel_rl: mass 0.4 -> 0.05; geometry collision cylinder length=0.04 radius=0.03; visual cylinder length=0.04 radius=0.03
- link wheel_rr: mass 0.4 -> 0.05; geometry collision cylinder length=0.04 radius=0.03; visual cylinder length=0.04 radius=0.03
Joints:
- added joint ballast_joint: type fixed, parent base_link, child ballast, origin xyz=0 0 0.16
- joint rope_attachment_joint: origin xyz=0.25 0 0 -> xyz=0.30 0 0
- joint wheel_fl_joint: origin xyz=0.18 0.20 -0.07 -> xyz=0.26 0.20 -0.07
- joint wheel_fr_joint: origin xyz=0.18 -0.20 -0.07 -> xyz=0.26 -0.20 -0.07
- joint wheel_rl_joint: origin xyz=-0.18 0.20 -0.07 -> xyz=-0.26 0.20 -0.07
- joint wheel_rr_joint: origin xyz=-0.18 -0.20 -0.07 -> xyz=-0.26 -0.20 -0.07
