Commit message: 修改为real urdf

File: imgo2_description/xacro/core.xacro (robot description, xacro)
@@ -57,9 +57,9 @@
     <link name="FL_HIP">
         <inertial>
-            <origin xyz="0.05776150 0.01631658 0.00001927"/>
-            <mass value="0.66982842"/>
-            <inertia ixx="0.00047165" ixy="-0.00002152" ixz="-0.00000604"
-                    iyy="0.00094023" iyz="0.00000025"
-                    izz="0.00063679"/>
+            <origin xyz="0.05502 0.01629 0.00008"/>
+            <mass value="0.66"/>
+            <inertia ixx="0.00048724823" ixy="-0.00002083480" ixz="-0.00000122317"
+                    iyy="0.00090893629" iyz="0.00000075580"
+                    izz="0.000577702"/>
         </inertial>
         <visual>
@@ -84,9 +84,9 @@
     <link name="FL_THIGH">
         <inertial>
-            <origin rpy="0.0 0.0 0.0" xyz="-0.00429543 0.04392351 -0.03236426"/>
-            <mass value="0.96995719"/>
-            <inertia ixx="0.00506421" ixy="0.00008162" ixz="-0.00034748"
-                    iyy="0.00527087" iyz="0.00062882"
-                    izz="0.00088197"/>
+            <origin rpy="0.0 0.0 0.0" xyz="-0.002105 0.044398 -0.032405"/>
+            <mass value="1.044"/>
+            <inertia ixx="0.005502341" ixy="0.000037296" ixz="0.000245651"
+                    iyy="0.005694337" iyz="0.000658207"
+                    izz="0.000950721"/>
         </inertial>
         <visual>
@@ -180,9 +180,9 @@
     <link name="FR_HIP">
         <inertial>
-            <origin xyz="0.05776150 -0.01631658 0.00001927"/>
-            <mass value="0.66982842"/>
-            <inertia ixx="0.00047165" ixy="0.00002152" ixz="-0.00000604"
-                    iyy="0.00094023" iyz="-0.00000025"
-                    izz="0.00063679"/>
+            <origin xyz="0.05502 -0.01629 -0.00008"/>
+            <mass value="0.66"/>
+            <inertia ixx="0.00048724823" ixy="0.00002083480" ixz="0.00000122317"
+                    iyy="0.00090893629" iyz="0.00000075580"
+                    izz="0.000577702"/>
         </inertial>
         <visual>
@@ -207,9 +207,9 @@
     <link name="FR_THIGH">
         <inertial>
-            <origin rpy="0.0 0.0 0.0" xyz="-0.00429543 -0.04392351 -0.03236426"/>
-            <mass value="0.96995719"/>
-            <inertia ixx="0.00506421" ixy="-0.00008162" ixz="-0.00034748"
-                    iyy="0.00527087" iyz="-0.00062882"
-                    izz="0.00088197"/>
+            <origin rpy="0.0 0.0 0.0" xyz="-0.002105 -0.044398 -0.032405"/>
+            <mass value="1.044"/>
+            <inertia ixx="0.005502341" ixy="-0.000037296" ixz="-0.000245651"
+                    iyy="0.005694337" iyz="-0.000658207"
+                    izz="0.000950721"/>
         </inertial>
         <visual>
@@ -303,9 +303,9 @@
      <link name="RL_HIP">
         <inertial>
-            <origin xyz="-0.05776150 0.01631658 0.00001927"/>
-            <mass value="0.66982842"/>
-            <inertia ixx="0.00047165" ixy="0.00002152" ixz="0.00000604"
-                    iyy="0.00094023" iyz="0.00000025"
-                    izz="0.00063679"/>
+            <origin xyz="-0.05502 0.01629 -0.00008"/>
+            <mass value="0.66"/>
+            <inertia ixx="0.00047490383" ixy="0.00002083480" ixz="-0.00000122317"
+                    iyy="0.00090893629" iyz="-0.00000075580"
+                    izz="0.000577702"/>
         </inertial>
         <visual>
@@ -330,9 +330,9 @@
     <link name="RL_THIGH">
         <inertial>
-            <origin rpy="0.0 0.0 0.0" xyz="0.00429543 0.04392351 -0.03236426"/>
-            <mass value="0.96995719"/>
-            <inertia ixx="0.00506421" ixy="0.00008162" ixz="-0.00034748"
-                    iyy="0.00527087" iyz="0.00062882"
-                    izz="0.00088197"/>
+            <origin rpy="0.0 0.0 0.0" xyz="-0.002105 0.044398 -0.032405"/>
+            <mass value="1.044"/>
+            <inertia ixx="0.005502341" ixy="0.000037296" ixz="0.000245651"
+                    iyy="0.005694337" iyz="0.000658207"
+                    izz="0.000950721"/>
         </inertial>
         <visual>
@@ -426,9 +426,9 @@
     <link name="RR_HIP">
         <inertial>
-            <origin xyz="-0.05776150 -0.01631658 0.00001927"/>
-            <mass value="0.66982842"/>
-            <inertia ixx="0.00047165" ixy="-0.00002152" ixz="0.00000604"
-                    iyy="0.00094023" iyz="-0.00000025"
-                    izz="0.00063679"/>
+            <origin xyz="-0.05502 -0.01629 0.00008"/>
+            <mass value="0.66"/>
+            <inertia ixx="0.00047490383" ixy="-0.00002083480" ixz="0.00000122317"
+                    iyy="0.00090893629" iyz="-0.00000075580"
+                    izz="0.000577702"/>
         </inertial>
         <visual>
@@ -453,9 +453,9 @@
     <link name="RR_THIGH">
         <inertial>
-            <origin rpy="0.0 0.0 0.0" xyz="0.00429543 -0.04392351 -0.03236426"/>
-            <mass value="0.96995719"/>
-            <inertia ixx="0.00506421" ixy="-0.00008162" ixz="-0.00034748"
-                    iyy="0.00527087" iyz="-0.00062882"
-                    izz="0.00088197"/>
+            <origin rpy="0.0 0.0 0.0" xyz="-0.002105 -0.044398 -0.032405"/>
+            <mass value="1.044"/>
+            <inertia ixx="0.005502341" ixy="-0.000037296" ixz="-0.000245651"
+                    iyy="0.005694337" iyz="-0.000658207"
+                    izz="0.000950721"/>
         </inertial>
         <visual>

Commit message: 修改了模型,更新了amp datasets, 并重新训练

File: imgo2_description/xacro/core.xacro (robot description, xacro)
@@ -86,5 +86,5 @@
             <origin rpy="0.0 0.0 0.0" xyz="-0.002105 0.044398 -0.032405"/>
             <mass value="1.044"/>
-            <inertia ixx="0.005502341" ixy="0.000037296" ixz="0.000245651"
+            <inertia ixx="0.005502341" ixy="0.000037296" ixz="-0.000245651"
                     iyy="0.005694337" iyz="0.000658207"
                     izz="0.000950721"/>
@@ -332,5 +332,5 @@
             <origin rpy="0.0 0.0 0.0" xyz="-0.002105 0.044398 -0.032405"/>
             <mass value="1.044"/>
-            <inertia ixx="0.005502341" ixy="0.000037296" ixz="0.000245651"
+            <inertia ixx="0.005502341" ixy="0.000037296" ixz="-0.000245651"
                     iyy="0.005694337" iyz="0.000658207"
                     izz="0.000950721"/>

Commit message: 修复历史合并引入的重复配置与资源回退

File: imgo2_description/xacro/core.xacro (robot description, xacro)
@@ -62,9 +62,4 @@
                     iyy="0.00090893629" iyz="0.00000075580"
                     izz="0.000577702"/>
-            <origin xyz="0.05502 0.01629 0.00008"/>
-            <mass value="0.66"/>
-            <inertia ixx="0.00048724823" ixy="-0.00002083480" ixz="-0.00000122317"
-                    iyy="0.00090893629" iyz="0.00000075580"
-                    izz="0.000577702"/>
         </inertial>
         <visual>
@@ -190,9 +185,4 @@
                     iyy="0.00090893629" iyz="0.00000075580"
                     izz="0.000577702"/>
-            <origin xyz="0.05502 -0.01629 -0.00008"/>
-            <mass value="0.66"/>
-            <inertia ixx="0.00048724823" ixy="0.00002083480" ixz="0.00000122317"
-                    iyy="0.00090893629" iyz="0.00000075580"
-                    izz="0.000577702"/>
         </inertial>
         <visual>
@@ -222,9 +212,4 @@
                     iyy="0.005694337" iyz="-0.000658207"
                     izz="0.000950721"/>
-            <origin rpy="0.0 0.0 0.0" xyz="-0.002105 -0.044398 -0.032405"/>
-            <mass value="1.044"/>
-            <inertia ixx="0.005502341" ixy="-0.000037296" ixz="-0.000245651"
-                    iyy="0.005694337" iyz="-0.000658207"
-                    izz="0.000950721"/>
         </inertial>
         <visual>
@@ -318,9 +303,4 @@
      <link name="RL_HIP">
         <inertial>
-            <origin xyz="-0.05502 0.01629 -0.00008"/>
-            <mass value="0.66"/>
-            <inertia ixx="0.00047490383" ixy="0.00002083480" ixz="-0.00000122317"
-                    iyy="0.00090893629" iyz="-0.00000075580"
-                    izz="0.000577702"/>
             <origin xyz="-0.05502 0.01629 -0.00008"/>
             <mass value="0.66"/>
@@ -451,9 +431,4 @@
                     iyy="0.00090893629" iyz="-0.00000075580"
                     izz="0.000577702"/>
-            <origin xyz="-0.05502 -0.01629 0.00008"/>
-            <mass value="0.66"/>
-            <inertia ixx="0.00047490383" ixy="-0.00002083480" ixz="0.00000122317"
-                    iyy="0.00090893629" iyz="-0.00000075580"
-                    izz="0.000577702"/>
         </inertial>
         <visual>
@@ -483,9 +458,4 @@
                     iyy="0.005694337" iyz="-0.000658207"
                     izz="0.000950721"/>
-            <origin rpy="0.0 0.0 0.0" xyz="-0.002105 -0.044398 -0.032405"/>
-            <mass value="1.044"/>
-            <inertia ixx="0.005502341" ixy="-0.000037296" ixz="-0.000245651"
-                    iyy="0.005694337" iyz="-0.000658207"
-                    izz="0.000950721"/>
         </inertial>
         <visual>
